File: DC36_DC5.kicad_sch (KiCad schematic)
At the start: 19 parts, among them U1 LM2596S

Commit message: Ver 1.0
Parts:
- R1, R2: now not fitted
- RV1: now fitted
Changed lines of the file:
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@@
 		(in_bom yes)
 		(on_board yes)
-		(dnp yes)
+		(dnp no)
 		(property "Reference" "RV1"
 			(at 148.336 38.1 0)
@@
 		(in_bom yes)
 		(on_board yes)
-		(dnp no)
+		(dnp yes)
 		(fields_autoplaced yes)
 		(property "Reference" "R2"
@@
 		(in_bom yes)
 		(on_board yes)
-		(dnp no)
+		(dnp yes)
 		(fields_autoplaced yes)
 		(property "Reference" "R1"
