File: DC36_DC5.kicad_sch (KiCad schematic)
At the start: 19 parts, among them U1 LM2596S

Commit message: Ver 1.0
Parts:
- RV1: now not fitted
- U1: footprint Package_TO_SOT_SMD:TO-263-5_TabPin3 -> DCDC:LM2596S
- renumbered C4 to C3, C5 to C4, C3 to C5, H4 to H3, H3 to H4, R2 to R1, R3 to R2, R1 to R3
Changed lines of the file:
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@@
 		(dnp no)
 		(fields_autoplaced yes)
-		(property "Reference" "H3"
+		(property "Reference" "H4"
 			(at 214.63 50.7999 90)
 			(effects
@@
 			(project "DC36_DC5"
 				(path "/b72e6314-4bbd-4fa4-856f-1f0e58b9b2bd"
-					(reference "H3")
+					(reference "H4")
 					(unit 1)
 				)
@@
 		(dnp no)
 		(fields_autoplaced yes)
-		(property "Reference" "H4"
+		(property "Reference" "H3"
 			(at 213.36 85.0899 90)
 			(effects
@@
 			(project "DC36_DC5"
 				(path "/b72e6314-4bbd-4fa4-856f-1f0e58b9b2bd"
-					(reference "H4")
+					(reference "H3")
 					(unit 1)
 				)
@@
 		(dnp no)
 		(fields_autoplaced yes)
-		(property "Reference" "C4"
+		(property "Reference" "C3"
 			(at 177.8 72.3899 0)
 			(effects
@@
 			(project "DC36_DC5"
 				(path "/b72e6314-4bbd-4fa4-856f-1f0e58b9b2bd"
-					(reference "C4")
+					(reference "C3")
 					(unit 1)
 				)
@@
 		(in_bom yes)
 		(on_board yes)
-		(dnp no)
+		(dnp yes)
 		(property "Reference" "RV1"
 			(at 148.336 38.1 0)
@@
 		(dnp no)
 		(fields_autoplaced yes)
-		(property "Reference" "R3"
+		(property "Reference" "R2"
 			(at 176.53 44.4499 0)
 			(effects
@@
 			(project "DC36_DC5"
 				(path "/b72e6314-4bbd-4fa4-856f-1f0e58b9b2bd"
-					(reference "R3")
+					(reference "R2")
 					(unit 1)
 				)
@@
 			)
 		)
-		(property "Footprint" "Package_TO_SOT_SMD:TO-263-5_TabPin3"
+		(property "Footprint" "DCDC:LM2596S"
 			(at 133.35 64.77 0)
 			(effects
@@
 		(dnp no)
 		(fields_autoplaced yes)
-		(property "Reference" "R1"
+		(property "Reference" "R3"
 			(at 203.2 63.4999 0)
 			(effects
@@
 			(project ""
 				(path "/b72e6314-4bbd-4fa4-856f-1f0e58b9b2bd"
-					(reference "R1")
+					(reference "R3")
 					(unit 1)
 				)
@@
 		(dnp no)
 		(fields_autoplaced yes)
-		(property "Reference" "C5"
+		(property "Reference" "C4"
 			(at 195.58 44.4499 0)
 			(effects
@@
 			(project "DC36_DC5"
 				(path "/b72e6314-4bbd-4fa4-856f-1f0e58b9b2bd"
-					(reference "C5")
+					(reference "C4")
 					(unit 1)
 				)
@@
 		(dnp no)
 		(fields_autoplaced yes)
-		(property "Reference" "C3"
+		(property "Reference" "C5"
 			(at 195.58 71.5009 0)
 			(effects
@@
 			(project "DC36_DC5"
 				(path "/b72e6314-4bbd-4fa4-856f-1f0e58b9b2bd"
-					(reference "C3")
+					(reference "C5")
 					(unit 1)
 				)
@@
 		(dnp no)
 		(fields_autoplaced yes)
-		(property "Reference" "R2"
+		(property "Reference" "R1"
 			(at 176.53 33.0199 0)
 			(effects
@@
 			(project "DC36_DC5"
 				(path "/b72e6314-4bbd-4fa4-856f-1f0e58b9b2bd"
-					(reference "R2")
-					(unit 1)
-				)
+					(reference "R1")
+					(unit 1)
+				)

Commit message: V1.01
Parts:
- added D4: SS56 60V/5A, Diode_SMD:D_SMB-SMC_Universal_Handsoldering, symbol Device:D_Schottky
- C4: value 180pF 50V -> 1200pF 50V; footprint Capacitor_SMD:C_0603_1608Metric -> Capacitor_SMD:C_1206_3216Metric
- R1, R2, R3: footprint Resistor_SMD:R_0603_1608Metric -> Resistor_SMD:R_0805_2012Metric_Pad1.20x1.40mm_HandSolder
Connections:
- net at C4.1, H4.1, R2.1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: now also D4.1 (K); no longer C3.1, C5.1, L1.2
- new net: C3.1, C5.1, D4.2 (A), L1.2
Other:
- moved on the sheet: C4, D3, R3

Commit message: Add dtscription
Parts:
- C1, C3: Platan SKU (none) -> 2014968057
- C2: Platan SKU (none) -> 2015341406
- C4: Platan SKU (none) -> 2014969669
- C5: Platan SKU (none) -> 403869617
- D1, D2: value STPS20M100SG -> SS520; Platan SKU (none) -> 2014859847
- D3: Platan SKU (none) -> 2015697923
- D4: value SS56 60V/5A -> SS520; Platan SKU (none) -> 2014859847
- F1: Platan SKU (none) -> 38409
- L1: Platan SKU (none) -> 2016862973
- R1: Platan SKU (none) -> 2010220531
- R2: Platan SKU (none) -> 2010018418
- R3: Platan SKU (none) -> 2014969702
- U1: Platan SKU (none) -> 344157231
Changed lines of the file:
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@@
+		)
+	)
+	(text_box "1. При установке подстроечного резистора RV1, не устанавливаются элементы поз. R1 R2 и наоборот.\n\n2. При использовании U1 в исполнении на фиксированное выходное напряжение, не устанавливаются\n элементы поз. R1, R2, RV1, C4, а на место R2 устанавливается перемычка.\n\n3. Посадочные места элементов D1, D2 допускают установку подходящих по параметрам диодов в корпусах\nDPAK, D2PAK, SMB, SMC; D4 - SMB, SMC.\n\n4. Посадочные места элементов С2, С5 - допускают установку подходящих по параметрам конденсаторов\nв корпусах 8 и 10 мм.\n\n5. Посадочное место L1 позволяет устанавливать дроссели типоразмеров от 10х10 до 18х18.\n\n"
+		(exclude_from_sim no)
+		(at 41.91 107.95 0)
+		(size 120.65 85.09)
+		(stroke
+			(width -0.0001)
+			(type default)
+		)
+		(fill
+			(type none)
+		)
+		(effects
+			(font
+				(face "KiCad Font")
+				(size 2.54 2.54)
+			)
+			(justify left top)
 		)
 	)
@@
 			)
 		)
-		(property "Value" "STPS20M100SG"
+		(property "Value" "SS520"
 			(at 152.4 73.3424 90)
 			(effects
@@
 			)
 		)
-		(property "Description" "Schottky diode"
+		(property "Description" "SS520, SMT выпрямительный диод Шоттки, 200В, 5А (DO-214AB (SMC))"
+			(at 149.86 72.39 0)
+			(effects
+				(font
+					(size 1.27 1.27)
+				)
+				(hide yes)
+			)
+		)
+		(property "Platan SKU" "2014859847 "
 			(at 149.86 72.39 0)
 			(effects
@@
 			)
 		)
-		(property "Description" "Light emitting diode"
+		(property "Description" "L-C170GCT, светодиод зеленый 12.5мКд SMD 0805"
+			(at 218.44 78.74 0)
+			(effects
+				(font
+					(size 1.27 1.27)
+				)
+				(hide yes)
+			)
+		)
+		(property "Platan SKU" "2015697923 "
 			(at 218.44 78.74 0)
 			(effects
@@
 			)
 		)
+		(property "Platan SKU" ""
+			(at 233.68 52.07 0)
+			(effects
+				(font
+					(size 1.27 1.27)
+				)
+				(hide yes)
+			)
+		)
 		(pin "1"
 		)
@@
 			)
 		)
+		(property "Platan SKU" ""
+			(at 232.41 86.36 0)
+			(effects
+				(font
+					(size 1.27 1.27)
+				)
+				(hide yes)
+			)
+		)
 		(pin "1"
 		)
@@
 			)
 		)
-		(property "Value" "STPS20M100SG"
+		(property "Value" "SS520"
 			(at 93.0275 52.07 0)
 			(effects
@@
 			)
 		)
-		(property "Description" "Schottky diode"
+		(property "Description" "SS520, SMT выпрямительный диод Шоттки, 200В, 5А (DO-214AB (SMC))"
+			(at 92.71 55.88 0)
+			(effects
+				(font
+					(size 1.27 1.27)
+				)
+				(hide yes)
+			)
+		)
+		(property "Platan SKU" "2014859847 "
 			(at 92.71 55.88 0)
 			(effects
@@
 			)
 		)
-		(property "Description" "Unpolarized capacitor"
+		(property "Description" "GRM188R60J106ME47D, Конденсаторы керамические"
+			(at 173.99 73.66 0)
+			(effects
+				(font
+					(size 1.27 1.27)
+				)
+				(hide yes)
+			)
+		)
+		(property "Platan SKU" "2014968057 "
 			(at 173.99 73.66 0)
 			(effects
@@
 			)
 		)
+		(property "Platan SKU" ""
+			(at 156.21 40.64 0)
+			(effects
+				(font
+					(size 1.27 1.27)
+				)
+				(hide yes)
+			)
+		)
 		(pin "2"
 		)
@@
 			)
 		)
-		(property "Description" "Polarized capacitor"
+		(property "Description" "EEHZA1H680P, SMD эл-лит 50V 68uF /8*10.2/105 C Polymer Hybrid"
+			(at 107.95 73.66 0)
+			(effects
+				(font
+					(size 1.27 1.27)
+				)
+				(hide yes)
+			)
+		)
+		(property "Platan SKU" "2015341406 "
 			(at 107.95 73.66 0)
 			(effects
@@
 			)
 		)
-		(property "Description" "Resettable fuse, polymeric positive temperature coefficient"
+		(property "Description" "MF-R300, 3.0A самовосстанавливающийся предохранитель"
+			(at 71.12 55.88 0)
+			(effects
+				(font
+					(size 1.27 1.27)
+				)
+				(hide yes)
+			)
+		)
+		(property "Platan SKU" "38409 "
 			(at 71.12 55.88 0)
 			(effects
@@
 			)
 		)
+		(property "Platan SKU" ""
+			(at 53.34 55.88 0)
+			(effects
+				(font
+					(size 1.27 1.27)
+				)
+				(hide yes)
+			)
+		)
 		(pin "1"
 		)
@@
 			)
 		)
-		(property "Description" "Resistor"
+		(property "Description" "RC0805FR-073K09L, 0805, чип 0805      3.09К 1%"
+			(at 173.99 45.72 0)
+			(effects
+				(font
+					(size 1.27 1.27)
+				)
+				(hide yes)
+			)
+		)
+		(property "Platan SKU" "2010018418 "
 			(at 173.99 45.72 0)
 			(effects
@@
 			)
 		)
-		(property "Description" "5V 3A Step-Down Voltage Regulator, TO-263"
+		(property "Description" "LM2596SX-ADJ, TO263-5"
+			(at 132.08 58.42 0)
+			(effects
+				(font
+					(size 1.27 1.27)
+				)
+				(hide yes)
+			)
+		)
+		(property "Platan SKU" "344157231 "
 			(at 132.08 58.42 0)
 			(effects
@@
 			)
 		)
+		(property "Platan SKU" ""
+			(at 53.34 86.36 0)
+			(effects
+				(font
+					(size 1.27 1.27)
+				)
+				(hide yes)
+			)
+		)
 		(pin "1"
 		)
@@
 			)
 		)
-		(property "Description" "Resistor"
+		(property "Description" "RC0805FR-07200RL, Резисторы постоянные"
+			(at 218.44 69.85 0)
+			(effects
+				(font
+					(size 1.27 1.27)
+				)
+				(hide yes)
+			)
+		)
+		(property "Platan SKU" "2014969702 "
 			(at 218.44 69.85 0)
 			(effects
@@
 			)
 		)
-		(property "Description" "Unpolarized capacitor"
+		(property "Description" "CC1206JRNPO9BN122, Конденсаторы керамические"
+			(at 184.15 46.99 0)
+			(effects
+				(font
+					(size 1.27 1.27)
+				)
+				(hide yes)
+			)
+		)
+		(property "Platan SKU" "2014969669 "
 			(at 184.15 46.99 0)
 			(effects
@@
 			)
 		)
-		(property "Description" "Inductor with ferrite core"
+		(property "Description" "IHLP6767DZER470M11, SMD 17.15*17.15*4"
+			(at 162.56 60.96 0)
+			(effects
+				(font
+					(size 1.27 1.27)
+				)
+				(hide yes)
+			)
+		)
+		(property "Platan SKU" "2016862973 "
 			(at 162.56 60.96 0)
 			(effects
@@
 			)
 		)
-		(property "Value" "SS56 60V/5A"
+		(property "Value" "SS520"
 			(at 204.7875 57.15 0)
 			(effects
@@
 			)
 		)
-		(property "Description" "Schottky diode"
+		(property "Description" "SS520, SMT выпрямительный диод Шоттки, 200В, 5А (DO-214AB (SMC))"
+			(at 204.47 60.96 0)
+			(effects
+				(font
+					(size 1.27 1.27)
+				)
+				(hide yes)
+			)
+		)
+		(property "Platan SKU" "2014859847 "
 			(at 204.47 60.96 0)
 			(effects
@@
 			)
 		)
-		(property "Description" "Polarized capacitor"
+		(property "Description" "EEEFK1V331P, ЧИП электролит.конд.  330мкф  35В 105гр,  10x10.2(G) 2т.ч"
+			(at 191.77 73.66 0)
+			(effects
+				(font
+					(size 1.27 1.27)
+				)
+				(hide yes)
+			)
+		)
+		(property "Platan SKU" "403869617 "
 			(at 191.77 73.66 0)
 			(effects
@@
 			)
 		)
-		(property "Description" "Unpolarized capacitor"
+		(property "Description" "GRM188R60J106ME47D, Конденсаторы керамические"
+			(at 82.55 73.66 0)
+			(effects
+				(font
+					(size 1.27 1.27)
+				)
+				(hide yes)
+			)
+		)
+		(property "Platan SKU" "2014968057 "
 			(at 82.55 73.66 0)
 			(effects
@@
 			)
 		)
-		(property "Description" "Resistor"
+		(property "Description" "CR0805-FX-1001ELF, чип резистор 0805 1кОм"
 			(at 173.99 34.29 0)
 			(effects
+				(font
+					(size 1.27 1.27)
+				)
+				(hide yes)
+			)
+		)
+		(property "Platan SKU" "2010220531 "
+			(at 173.99 34.29 0)
+			(effects
