File: DC36_DC5.kicad_pcb (KiCad board)
At the start: 2 copper layers, 69 x 39 mm, 20 parts, among them U1 LM2596S

Commit message: Ver 1.0
Parts:
- added ARROW: ARROW, DCDC:ARROW, F.Cu at (127.4, 112.5)
- U1: footprint Package_TO_SOT_SMD:TO-263-5_TabPin3 -> DCDC:LM2596S
- moved C1 5.85 mm to (102.2, 92.9), turned to 180 degrees
- moved D3 4.69 mm to (150.4, 97.4)
- moved F1 4.41 mm to (98.2, 93.3)
- moved C3 3.92 mm to (134.4, 87.3)
- moved C2 1.84 mm to (106.9, 85.4)
- moved D1 1.50 mm to (105.6, 104.8)
- moved RV1 1.00 mm to (115.2, 106.7)
- renumbered C4 to C3, C5 to C4, C3 to C5, H4 to H3, H3 to H4, R2 to R1, R3 to R2, R1 to R3
Routing:
- net P,GND: track 25.4 -> 6.10 mm, vias 9 -> 28
- net Net-(D1-A): track 16.6 -> 9.41 mm
- net Net-(U1-FB): track 29.6 -> 23.8 mm
- net Net-(D3-A): track 6.35 -> 4.47 mm
- net Net-(F1-Pad1): track 12.0 -> 13.3 mm
- net Net-(D2-K): track 46.4 -> 45.3 mm
- net Net-(C3-Pad1): track 92.3 -> 91.5 mm
- net Net-(D1-K): track 41.2 -> 41.7 mm
Other:
- board text added: "1"
- board text added: "2"
- board text added: "3"
- board text added: "4"
- board text added: "5 V"
- board text added: "6-36 V"

Commit message: V1.01
Parts:
- added D4: SS56 60V/5A, Diode_SMD:D_SMB-SMC_Universal_Handsoldering, F.Cu at (141.1, 80.6)
- C4: value 180pF 50V -> 1200pF 50V; footprint Capacitor_SMD:C_0603_1608Metric -> Capacitor_SMD:C_1206_3216Metric
- R1, R2, R3: footprint Resistor_SMD:R_0603_1608Metric -> Resistor_SMD:R_0805_2012Metric_Pad1.20x1.40mm_HandSolder
- moved C3 22.0 mm to (112.8, 83.2), turned to 90 degrees
- moved C5 3.06 mm to (141.9, 89.8), turned to 0 degrees
- moved D2 1.96 mm to (142.8, 102.0)
- moved C2 1.64 mm to (105.3, 85.0)
- moved L1 0.64 mm to (123.3, 87.4)
Connections:
- C3 pad 1: Net-(C3-Pad1) -> Net-(D4-A)
- C4 pad 1: Net-(C3-Pad1) -> Net-(D4-K)
- C5 pad 1: Net-(C3-Pad1) -> Net-(D4-A)
- H4 pad 1: Net-(C3-Pad1) -> Net-(D4-K)
- L1 pad 2: Net-(C3-Pad1) -> Net-(D4-A)
- R2 pad 1: Net-(C3-Pad1) -> Net-(D4-K)
- R3 pad 1: Net-(C3-Pad1) -> Net-(D4-K)
- RV1 pad 3: Net-(C3-Pad1) -> Net-(D4-K)
Routing:
- net Net-(C3-Pad1): track 91.5 -> 0.00 mm, vias 1 -> 0
- net Net-(D4-K): track 0.00 -> 78.1 mm, vias 0 -> 1
- net Net-(D4-A): track 0.00 -> 39.2 mm
- net Net-(D1-K): track 41.7 -> 42.6 mm
- net Net-(D2-K): track 45.3 -> 44.7 mm
- net P,GND: vias 28 -> 25
Other:
- board text added: "V1.01 22.10.24"
