File: DC36_DC5.kicad_pcb (KiCad board)
At the start: 2 copper layers, 69 x 39 mm, 22 parts, among them U1 LM2596S

Commit message: To prod
Parts:
- removed LOGO: LOGO, DCDC:LOGO
- added G***: LOGO1, DCDC:LOGO1, F.Cu at (111.8, 92.0)
